Commit message: fix: edit path, add composer example

File: urdf/rm_65_b.urdf (robot description, URDF)
Before this commit: robot rm_65_b, 8 links, 7 joints
Links:
- link Link1: geometry collision mesh filename=/home/simt-wj/01_Active/tesseract_python/meshes/rm_65_b/lin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; visual mesh filename=/home/simt-wj/01_Active/tesseract_python/meshes/rm_65_b/lin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
- link Link2: geometry collision mesh filename=/home/simt-wj/01_Active/tesseract_python/meshes/rm_65_b/lin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; visual mesh filename=/home/simt-wj/01_Active/tesseract_python/meshes/rm_65_b/lin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
- link Link3: geometry collision mesh filename=/home/simt-wj/01_Active/tesseract_python/meshes/rm_65_b/lin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; visual mesh filename=/home/simt-wj/01_Active/tesseract_python/meshes/rm_65_b/lin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
- link Link4: geometry collision mesh filename=/home/simt-wj/01_Active/tesseract_python/meshes/rm_65_b/lin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; visual mesh filename=/home/simt-wj/01_Active/tesseract_python/meshes/rm_65_b/lin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
- link Link5: geometry collision mesh filename=/home/simt-wj/01_Active/tesseract_python/meshes/rm_65_b/lin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; visual mesh filename=/home/simt-wj/01_Active/tesseract_python/meshes/rm_65_b/lin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
- link Link6: geometry collision mesh filename=/home/simt-wj/01_Active/tesseract_python/meshes/rm_65_b/lin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; visual mesh filename=/home/simt-wj/01_Active/tesseract_python/meshes/rm_65_b/lin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
- link base_link: geometry collision mesh filename=/home/simt-wj/01_Active/tesseract_python/meshes/rm_65_b/bas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; visual mesh filename=/home/simt-wj/01_Active/tesseract_python/meshes/rm_65_b/bas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

Commit message: feat: added dummy gripper and tcp for planning, tested planning around obstacles

File: urdf/rm_65_b.urdf (robot description, URDF)
Before this commit: robot rm_65_b, 8 links, 7 joints
Links:
- added link dummy_gripper, mass 0.1; collision cylinder length=0.2 radius=0.06; visual cylinder length=0.2 radius=0.06
- added link dummy_tcp, mass 0.7; collision box size=0.05 0.05 0.05; visual box size=0.01 0.01 0.01
Joints:
- added joint joint_gripper_fixed: type fixed, parent Link6, child dummy_gripper, origin xyz=0 0 0.11 rpy=0 0 0
- added joint joint_tcp_fixed: type fixed, parent dummy_gripper, child dummy_tcp, origin xyz=0 0 0.11 rpy=0 0 0
