Commit message: feat: update urdf

File: urdf/rm_65_b_full.urdf (robot description, URDF)
Before this commit: robot rm_65_b, 19 links, 18 joints
Links:
- added link camera_mount_link; collision box size=0.01 0.06 0.05; collision box size=0.09 0.06 0.01
- added link camera_plug_link; collision mesh filename=/home/simt-wj/01_Active/tesseract_python/meshes/realsense_d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; visual mesh filename=/home/simt-wj/01_Active/tesseract_python/meshes/realsense_d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
- added link gripper_mount_link; collision cylinder length=0.06 radius=0.039; visual cylinder length=0.06 radius=0.039
- link Link1: geometry collision mesh filename=/home/simt-wj/01_Active/tesseract_python/meshes/rm_65_b/lin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; visual mesh filename=/home/simt-wj/01_Active/tesseract_python/meshes/rm_65_b/lin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
- link Link2: geometry collision mesh filename=/home/simt-wj/01_Active/tesseract_python/meshes/rm_65_b/lin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; visual mesh filename=/home/simt-wj/01_Active/tesseract_python/meshes/rm_65_b/lin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
- link Link3: geometry collision mesh filename=/home/simt-wj/01_Active/tesseract_python/meshes/rm_65_b/lin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; visual mesh filename=/home/simt-wj/01_Active/tesseract_python/meshes/rm_65_b/lin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
- link Link4: geometry collision mesh filename=/home/simt-wj/01_Active/tesseract_python/meshes/rm_65_b/lin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; visual mesh filename=/home/simt-wj/01_Active/tesseract_python/meshes/rm_65_b/lin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
- link Link5: geometry collision mesh filename=/home/simt-wj/01_Active/tesseract_python/meshes/rm_65_b/lin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; visual mesh filename=/home/simt-wj/01_Active/tesseract_python/meshes/rm_65_b/lin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
- link Link6: geometry collision mesh filename=/home/simt-wj/01_Active/tesseract_python/meshes/rm_65_b/lin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; visual mesh filename=/home/simt-wj/01_Active/tesseract_python/meshes/rm_65_b/lin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
- link base_link: geometry collision mesh filename=/home/simt-wj/01_Active/tesseract_python/meshes/rm_65_b/bas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; visual mesh filename=/home/simt-wj/01_Active/tesseract_python/meshes/rm_65_b/bas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
- link camera_link: geometry collision box size=0.09 0.025 0.030; visual mesh filename=/home/simt-wj/01_Active/tesseract_python/meshes/realsense_d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
Joints:
- added joint camera_mount_joint: type fixed, parent Link6, child camera_mount_link, origin xyz=-0.055 0 0.035 rpy=0 0 0
- added joint camera_plug_joint: type fixed, parent camera_link, child camera_plug_link, origin xyz=-0.039 0. -0.021 rpy=0 1.57 -1.57
- added joint gripper_mount_joint: type fixed, parent Link6, child gripper_mount_link, origin xyz=0 0 0.03 rpy=0 0 0
- joint camera_joint: origin xyz=-0.11 0.00 0.07 rpy=0.4 0.0 1.57 -> xyz=-0.055 0 0.035 rpy=0.39 0.0 1.57; parent Link6 -> camera_mount_link
- joint joint_tcp_fixed: origin xyz=0 0 0.063 rpy=0 0 1.5708 -> xyz=0 0 0.033 rpy=0 0 1.5708; parent Link6 -> gripper_mount_link

Commit message: urdf: update visual and collision properties for camera and associated links

File: urdf/rm_65_b_full.urdf (robot description, URDF)
Before this commit: robot rm_65_b, 22 links, 21 joints
Links:
- link camera_mount_link: geometry collision box size=0.08 0.06 0.01; collision box size=0.1 0.08 0.01
Joints:
- joint camera_joint: origin xyz=-0.055 0 0.035 rpy=0.39 0.0 1.57 -> xyz=-0.0647 0 0.0346 rpy=0.249268 -0.009838 1.584086
